File: led_driver.sch (KiCad schematic (older format))
At the start: 27 parts, among them P1 PIN, T1 MOSFET, T2 MOSFET, T3 MOSFET, T4 MOSFET, T5 MOSFET, T6 MOSFET, U1 Teensy_3.1

Commit message: added schematic print. Produced GERBER files (manufacturing drawings). Slight rewiring to give larger passage ways for higher current flow
Other:
- note added: "1.0\n"
- note added: "Author: Denis Draca\nCommision: Marc Charmichael (UTS:CAS)"
- note added: "MMD Sawyer Base LED Driver Circuit"
- moved on the sheet: RGB1

Commit message: added DC jack, added 3d models for the RGB connectors and opamps
Parts:
- P1: footprint PIN:PIN -> Connectors:BARREL_JACK
Changed lines of the file:
@@
 F 0 "P1" H 5750 6900 60  0000 C CNN
 F 1 "PIN" H 5750 7200 60  0000 C CNN
-F 2 "PIN:PIN" H 5350 7050 60  0001 C CNN
+F 2 "Connectors:BARREL_JACK" H 5350 7050 60  0001 C CNN
 F 3 "~" H 5350 7050 60  0000 C CNN
 	1    5350 7050
